File: creatureControl/CreatureControl5x12-1.2.kicad_sch (KiCad schematic)
At the start: 49 parts, among them J1 USB_C_Receptacle_PowerOnly_6P, J10 Conn_01x02_Socket, J12 Conn_01x05_Pin, J2 Barrel_Jack, J3 Screw_Terminal_01x02, J4 Conn_01x03_Socket, J5 Conn_01x03_Socket, J6 Conn_01x03_Socket, J7 Conn_01x03_Socket, J8 Conn_01x05_Socket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

Commit message: Update board files to version 1.2
Parts:
- removed C1: 1000µF, symbol Device:C
- removed C2, C3, C4, C5, C6: 100µF, symbol Device:C
- removed SRV3: Conn_01x03_Pin, symbol Connector:Conn_01x03_Pin
- added C1: 1000µF, symbol Device:C_Polarized_US
- added C10: 1µF, symbol Device:C
- added C11: 220µF, symbol Device:C_Polarized_US
- added C12: 100nF, symbol Device:C
- added C2, C3, C4, C5, C6: 100µF, symbol Device:C_Polarized_US
- added SRV1: Conn_01x03_Pin, symbol Connector:Conn_01x03_Pin
- C7, C8: value 1µF -> 0.1µF
- renumbered SRV1 to SRV3
Connections:
- net +3V3: no longer C9.2, U3.1 (VCC)
- net +5V: now also C9.2, U3.1 (VCC), C1.1, C10.2, C11.1, C12.2, C2.1, C3.1, C4.1, C5.1, C6.1, SRV1.2 (Pin_2)
- net GND: now also C1.2, C10.1, C11.2, C12.1, C2.2, C3.2, C4.2, C5.2, C6.2, SRV1.1 (Pin_1)
- net at SRV3.3 (Pin_3): now also MCU1.6 (GP27); no longer MCU1.12 (GP2)
- net at J12.3 (Pin_3): now also MCU1.14 (GP4); no longer MCU1.6 (GP27)
- net at J12.4 (Pin_4): now also MCU1.13 (GP3); no longer MCU1.5 (GP28)
- net at J12.5 (Pin_5): now also MCU1.12 (GP2); no longer MCU1.4 (GP29)
- net at SRV2.3 (Pin_3): now also MCU1.5 (GP28); no longer MCU1.13 (GP3)
- new net: MCU1.4 (GP29), SRV1.3 (Pin_3)
Other:
- moved on the sheet: C7, C8, C9, D1, D2, J1, J2, J3, LED1, LED2, M1, M2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
