File: creatureControl/CreatureControl5x12-1.2.kicad_pcb (KiCad board)
At the start: 2 copper layers, 120 x 50 mm, 44 parts, among them J1 USB_C_Receptacle_GCT_USB4125-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, J2 BarrelJack_Horizontal, J3 TerminalBlock_4Ucon_1x02_P3.5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

Commit message: Update board files to version 1.2
Parts:
- added C10: C_Disc_D5.0mm_W2.5mm_P5.00mm, Capacitor_THT:C_Disc_D5.0mm_W2.5mm_P5.00mm, F.Cu at (109.2, 55.7)
- added C11: CP_Radial_D5.0mm_P2.50mm, Capacitor_THT:CP_Radial_D5.0mm_P2.50mm, F.Cu at (113.8, 55.6)
- added C12: C_Disc_D5.0mm_W2.5mm_P5.00mm, Capacitor_THT:C_Disc_D5.0mm_W2.5mm_P5.00mm, F.Cu at (185.6, 44.0)
- moved G*** 31.4 mm to (121.2, 50.6)
- moved G*** 23.6 mm to (153.7, 43.3)
- moved C9 20.0 mm to (105.8, 55.7)
- moved G*** 7.71 mm to (114.3, 69.5)
- moved SPKR 5.14 mm to (99.1, 72.4), turned to 0 degrees
- moved C1 3.43 mm to (181.0, 42.1)
- moved G*** 2.37 mm to (134.1, 66.5)
- moved R6 2.26 mm to (172.8, 76.3)
- moved C8 1.64 mm to (146.2, 48.6)
- moved C7 1.64 mm to (168.3, 48.6)
- moved DFPlayer Mini 1.63 mm to (114.6, 67.3), turned to 0 degrees
- moved R1 1.43 mm to (174.9, 57.1)
- moved R2 0.98 mm to (171.8, 53.9)
Connections:
- C9 pad 1: 3V3 -> 5V
- DFPlayer Mini pad 1: 3V3 -> 5V
- REF** pad 3: GP27 -> GP2
- REF** pad 4: GP28 -> GP3
- REF** pad 5: GP29 -> GP4
- SRV1 pad 1: GP2 -> GP29
- SRV2 pad 1: GP3 -> GP28
- SRV3 pad 1: GP4 -> GP27
Routing:
- net GP4: track 126.6 -> 47.0 mm, vias 1 -> 0
- net GP3: track 115.6 -> 53.3 mm, vias 1 -> 0
- net GP2: track 110.9 -> 60.5 mm, vias 1 -> 0
- net GP27: track 55.3 -> 104.4 mm, vias 0 -> 1
- net GP28: track 54.5 -> 93.8 mm, vias 0 -> 1
- net GP29: track 53.9 -> 90.9 mm, vias 0 -> 1
- net 3V3: track 82.6 -> 45.8 mm
- net 5V: track 245.5 -> 272.2 mm
- net GND: track 25.7 -> 48.4 mm, vias 18 -> 28
- net SPKR+: track 23.3 -> 7.15 mm
- net SPKR-: track 22.2 -> 7.15 mm
- net DFRX: track 55.1 -> 65.9 mm, vias 1 -> 0
- net GP1: track 85.4 -> 94.9 mm, vias 0 -> 1
- net GP13: track 97.0 -> 100.0 mm
- net GP0: track 27.1 -> 24.3 mm
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Other:
- board text added: "5V.GND.GP2.GP3.GP4"
- board text added: "5X12 v.1.2"
- board text added: "GP27"
- board text added: "GP28"
- board text added: "GP29"
- board text removed: "5V.GND.GP27.28.29"
- board text removed: "5X12 v.1.1"
- board text removed: "GP2"
- board text removed: "GP3"
- board text removed: "GP4"

Commit message: Upgrade bottoms silkscreen art
Parts:
- removed the G*** at (105.2, 46.6)
- added G***: LOGO, CreatureControl:HalloweenMoon, B.Cu at (152.6, 42.7)
- added G***: LOGO, CreatureControl:GraveyardLeft, B.Cu at (167.1, 66.0)
- added G***: LOGO, CreatureControl:GraveyardRight, B.Cu at (135.6, 68.8)
- added G***: LOGO, CreatureControl:Bats02, B.Cu at (118.5, 45.3)
